Commit message: chore: clean up files
Signed-off-by: Kenji Miyake <kenji.miyake@tier4.jp>

File: sample_sensor_kit_description/urdf/sensor_kit.xacro (robot description, xacro)
@@ -2,10 +2,8 @@
 <robot xmlns:xacro="http://ros.org/wiki/xacro">
   <xacro:macro name="sensor_kit_macro" params="parent x y z roll pitch yaw">
-    <xacro:include filename="$(find velodyne_description)/urdf/HDL-32E.urdf.xacro"/>
     <xacro:include filename="$(find velodyne_description)/urdf/VLP-16.urdf.xacro"/>
     <xacro:include filename="$(find vls_description)/urdf/VLS-128.urdf.xacro"/>
     <xacro:include filename="$(find camera_description)/urdf/monocular_camera.xacro"/>
     <xacro:include filename="$(find imu_description)/urdf/imu.xacro"/>
-    <!-- <xacro:property name="pi" value="3.1415926835897931"/> -->
     <xacro:arg name="gpu" default="false"/>
     <xacro:arg name="config_dir" default="$(find sample_sensor_kit_description)/config"/>

File: sample_sensor_kit_description/urdf/sensors.xacro (robot description, xacro)
@@ -33,24 +33,3 @@
     />
   </xacro:VLP-16>
-  <xacro:include filename="$(find livox_description)/urdf/livox_horizon.xacro"/>
-  <xacro:livox_horizon_macro
-    name="livox_front_left"
-    parent="base_link"
-    x="${calibration['base_link']['livox_front_left_base_link']['x']}"
-    y="${calibration['base_link']['livox_front_left_base_link']['y']}"
-    z="${calibration['base_link']['livox_front_left_base_link']['z']}"
-    roll="${calibration['base_link']['livox_front_left_base_link']['roll']}"
-    pitch="${calibration['base_link']['livox_front_left_base_link']['pitch']}"
-    yaw="${calibration['base_link']['livox_front_left_base_link']['yaw']}"
-  />
-  <xacro:livox_horizon_macro
-    name="livox_front_right"
-    parent="base_link"
-    x="${calibration['base_link']['livox_front_right_base_link']['x']}"
-    y="${calibration['base_link']['livox_front_right_base_link']['y']}"
-    z="${calibration['base_link']['livox_front_right_base_link']['z']}"
-    roll="${calibration['base_link']['livox_front_right_base_link']['roll']}"
-    pitch="${calibration['base_link']['livox_front_right_base_link']['pitch']}"
-    yaw="${calibration['base_link']['livox_front_right_base_link']['yaw']}"
-  />
 </robot>
